File: Airband Scanner.kicad_sch (KiCad schematic)
At the start: 37 parts, among them J1 Antenna, J2 AudioJack3, Q1 2SC3355, Q2 BF256B, U1 NE612, U2 MC1350, U5 MC1350, Y2 Resonator, Y3 Resonator

Commit message: Add files via upload
Parts:
- removed R6: 10k, Resistor_THT:R_Axial_DIN0204_L3.6mm_D1.6mm_P2.54mm_Vertical, symbol Device:R
- added C17: 1uF, Capacitor_THT:CP_Radial_D5.0mm_P2.50mm, symbol Device:C_Small
- added C18, C19: 3-18pF, symbol Device:C_Trim
- added Q3: 2N3904, Package_TO_SOT_THT:TO-92_Inline, symbol Transistor_BJT:2N3904
- added R11: 10k, Resistor_THT:R_Axial_DIN0204_L3.6mm_D1.6mm_P2.54mm_Vertical, symbol Device:R
- R7: value 1k -> 10k
- Y2, Y3: value Resonator -> Murata SFE10.7MFP
Connections:
- net Control and DDS/5V: now also C13.1, C6.1, L3.1, L4.1, Q2.3 (D), R2.1, U1.8 (Vcc), U2.1 (Out_a), U2.2 (Vcc), U5.1 (Out_a), U5.2 (Vcc), C18.1, C19.1
- net Control and DDS/GND: now also C10.2, C14.2, C2.1, C7.2, C8.2, J1.2 (Ext), J2.S, Q1.2 (E), R10.1, R3.2, R4.1, R5.2, U1.3 (GND), U2.7 (GND), U5.3 (GND), Y2.2, Y3.2, Q3.1 (E)
- net Control and DDS/LO_clean: now also U1.6 (Osc_b)
- net at C13.2, C9.1, L4.2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: now also C19.2
- net Control and DDS/Audio Monitor In: now reaches C10.1, C11.1, Q2.2 (S), R5.1
- net at J2.T: now also C17.2; no longer R7.2
- net at C12.1, C6.2, L3.2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: now also C18.2
- net Control and DDS/AGC Out: now reaches R9.1
- net Control and DDS/AGC Out: now also R8.1
- net at R7.1: now also C17.1, Q3.3 (C); no longer C11.2
- new net: C11.2, R7.2
- new net: Q3.2 (B), R11.1
- new net Control and DDS/Squelch Out: R11.2
Other:
- sheet Control and DDS ports: added AGC Out, Audio Monitor In, Squelch Out; removed none
- note added: "Pin 1 Zin = 1500//3pF"
- note added: "Pin 4 Zin = 2k ohms"
- note added: "Squelch gate"
- note removed: "Pin 1 Zi = 1500//3pF"
- note removed: "Pin 4 Zi = 2k ohms"
- title: (none) -> G1OJS Airband Scanner ATTiny85 Si5351 Project
- moved on the sheet: J2, R8, R9
